File: usb2ps2.kicad_sch (KiCad schematic)
At the start: 44 parts, among them CN1 USB, CN2 PS/2, CN3 UART, SW1 Flash Button, SW2 Reset Button, U1 W25Q128JVS, U2 NCP1117-3.3_SOT223, U3 RP2040, Y1 ABM8-272-T3

Commit message: HW Rev 1.0
Parts:
- renumbered C3 to C1, C14 to C10, C15 to C11, C16 to C12, C17 to C13, C18 to C14, C9 to C15, C12 to C16, C4 to C17, C5 to C18, C7 to C2, C10 to C3, C1 to C4, C2 to C5, C8 to C7, C11 to C8, C13 to C9, CN3 to CN2, CN2 to CN3, R3 to R1, R4 to R2, R2 to R3, R7 to R4, R8 to R6, R6 to R7, R9 to R8, R1 to R9, U2 to U1, U1 to U2
Other:
- moved on the sheet: C4, C5, CN3, L1, L2, PS1, R3, R5, R7, Y1

Commit message: HW Rev. 1.1
Connections:
- net +3V3: no longer R9.1, U2.1 (~{CS}), U3.56 (QSPI_SS)
- net GND: now also SW2.2; no longer SW2.3
- net RUN: now also SW2.3; no longer SW2.2
- new net QSPI_SS: R9.1, U2.1 (~{CS}), U3.56 (QSPI_SS)
Changed lines of the file:
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@@
 	(title_block
 		(title "USB to PS/2 Adapter")
-		(date "2024-10-25")
-		(rev "1.0")
+		(date "2024-11-13")
+		(rev "1.1")
 		(company "Mikhail Matveev")
 	)
@@
 	)
 	(junction
-		(at 97.79 105.41)
-		(diameter 0)
-		(color 0 0 0 0)
-	)
-	(junction
 		(at 177.8 76.2)
 		(diameter 0)
@@
 	)
 	(junction
-		(at 77.47 168.91)
+		(at 68.58 176.53)
 		(diameter 0)
 		(color 0 0 0 0)
@@
 	)
 	(junction
-		(at 63.5 125.73)
-		(diameter 0)
-		(color 0 0 0 0)
-	)
-	(junction
 		(at 196.85 81.28)
 		(diameter 0)
@@
 	)
 	(junction
-		(at 59.69 168.91)
+		(at 68.58 161.29)
 		(diameter 0)
 		(color 0 0 0 0)
@@
 	(wire
 		(pts
-			(xy 97.79 101.6) (xy 97.79 105.41)
+			(xy 97.79 101.6) (xy 97.79 120.65)
 		)
 		(stroke
@@
 	(wire
 		(pts
-			(xy 73.66 171.45) (xy 77.47 171.45)
-		)
-		(stroke
-			(width 0)
-			(type default)
-		)
-	)
-	(wire
-		(pts
 			(xy 229.87 104.14) (xy 241.3 104.14)
 		)
@@
 	(wire
 		(pts
-			(xy 59.69 171.45) (xy 63.5 171.45)
-		)
-		(stroke
-			(width 0)
-			(type default)
-		)
-	)
-	(wire
-		(pts
 			(xy 229.87 111.76) (xy 245.11 111.76)
 		)
@@
 	(wire
 		(pts
-			(xy 59.69 166.37) (xy 59.69 168.91)
+			(xy 68.58 161.29) (xy 73.66 161.29)
 		)
 		(stroke
@@
 	(wire
 		(pts
+			(xy 73.66 161.29) (xy 73.66 166.37)
+		)
+		(stroke
+			(width 0)
+			(type default)
+		)
+	)
+	(wire
+		(pts
 			(xy 189.23 81.28) (xy 194.31 81.28)
 		)
@@
 	(wire
 		(pts
+			(xy 63.5 161.29) (xy 68.58 161.29)
+		)
+		(stroke
+			(width 0)
+			(type default)
+		)
+	)
+	(wire
+		(pts
 			(xy 157.48 69.85) (xy 157.48 71.12)
 		)
@@
 	(wire
 		(pts
-			(xy 57.15 168.91) (xy 59.69 168.91)
+			(xy 68.58 158.75) (xy 68.58 161.29)
 		)
 		(stroke
@@
 	(wire
 		(pts
-			(xy 59.69 168.91) (xy 59.69 171.45)
-		)
-		(stroke
-			(width 0)
-			(type default)
-		)
-	)
-	(wire
-		(pts
-			(xy 52.07 125.73) (xy 63.5 125.73)
+			(xy 52.07 125.73) (xy 87.63 125.73)
 		)
 		(stroke
@@
 	(wire
 		(pts
-			(xy 77.47 168.91) (xy 77.47 171.45)
-		)
-		(stroke
-			(width 0)
-			(type default)
-		)
-	)
-	(wire
-		(pts
 			(xy 185.42 195.58) (xy 185.42 198.12)
 		)
@@
 	(wire
 		(pts
+			(xy 63.5 161.29) (xy 63.5 166.37)
+		)
+		(stroke
+			(width 0)
+			(type default)
+		)
+	)
+	(wire
+		(pts
 			(xy 248.92 104.14) (xy 262.89 104.14)
 		)
@@
 	(wire
 		(pts
-			(xy 229.87 144.78) (xy 245.11 144.78)
+			(xy 63.5 171.45) (xy 63.5 176.53)
 		)
 		(stroke
@@
 	(wire
 		(pts
-			(xy 280.67 72.39) (xy 269.24 72.39)
+			(xy 229.87 144.78) (xy 245.11 144.78)
 		)
 		(stroke
@@
 	(wire
 		(pts
-			(xy 73.66 166.37) (xy 77.47 166.37)
+			(xy 280.67 72.39) (xy 269.24 72.39)
 		)
 		(stroke
@@
 	(wire
 		(pts
-			(xy 104.14 102.87) (xy 104.14 101.6)
+			(xy 73.66 171.45) (xy 73.66 176.53)
 		)
 		(stroke
@@
 	(wire
 		(pts
-			(xy 269.24 72.39) (xy 257.81 72.39)
+			(xy 104.14 102.87) (xy 104.14 101.6)
 		)
 		(stroke
@@
 	(wire
 		(pts
-			(xy 63.5 166.37) (xy 59.69 166.37)
+			(xy 269.24 72.39) (xy 257.81 72.39)
 		)
 		(stroke
@@
 	(wire
 		(pts
-			(xy 63.5 125.73) (xy 87.63 125.73)
+			(xy 194.31 93.98) (xy 194.31 81.28)
 		)
 		(stroke
@@
 	(wire
 		(pts
-			(xy 194.31 93.98) (xy 194.31 81.28)
+			(xy 144.78 29.21) (xy 152.4 29.21)
 		)
 		(stroke
@@
 	(wire
 		(pts
-			(xy 144.78 29.21) (xy 152.4 29.21)
+			(xy 80.01 62.23) (xy 91.44 62.23)
 		)
 		(stroke
@@
 	(wire
 		(pts
-			(xy 80.01 62.23) (xy 91.44 62.23)
+			(xy 327.66 195.58) (xy 339.09 195.58)
 		)
 		(stroke
@@
 	(wire
 		(pts
-			(xy 327.66 195.58) (xy 339.09 195.58)
+			(xy 63.5 176.53) (xy 68.58 176.53)
 		)
 		(stroke
@@
 	(wire
 		(pts
-			(xy 77.47 166.37) (xy 77.47 168.91)
+			(xy 68.58 176.53) (xy 73.66 176.53)
 		)
 		(stroke
@@
 	(wire
 		(pts
-			(xy 77.47 168.91) (xy 81.28 168.91)
+			(xy 68.58 176.53) (xy 68.58 180.34)
 		)
 		(stroke
@@
 	(wire
 		(pts
-			(xy 63.5 105.41) (xy 63.5 125.73)
-		)
-		(stroke
-			(width 0)
-			(type default)
-		)
-	)
-	(wire
-		(pts
-			(xy 63.5 105.41) (xy 97.79 105.41)
-		)
-		(stroke
-			(width 0)
-			(type default)
-		)
-	)
-	(wire
-		(pts
 			(xy 198.12 29.21) (xy 198.12 27.94)
 		)
@@
 	(wire
 		(pts
-			(xy 97.79 105.41) (xy 97.79 120.65)
-		)
-		(stroke
-			(width 0)
-			(type default)
-		)
-	)
-	(wire
-		(pts
 			(xy 351.79 53.34) (xy 383.54 53.34)
 		)
@@
 	)
 	(label "RUN"
-		(at 81.28 168.91 0)
+		(at 68.58 180.34 270)
 		(fields_autoplaced yes)
 		(effects
@@
 				(size 1.27 1.27)
 			)
-			(justify left bottom)
+			(justify right bottom)
 		)
 	)
@@
 		(lib_name "GND_1")
 		(lib_id "power:GND")
-		(at 57.15 168.91 270)
+		(at 68.58 158.75 180)
 		(unit 1)
 		(exclude_from_sim no)
@@
 		(fields_autoplaced yes)
 		(property "Reference" "#PWR030"
-			(at 50.8 168.91 0)
+			(at 68.58 152.4 0)
 			(effects
 				(font
@@
 		)
 		(property "Value" "GND"
-			(at 53.34 168.9099 90)
+			(at 68.5801 154.94 90)
 			(effects
 				(font
@@
 		)
 		(property "Footprint" ""
-			(at 57.15 168.91 0)
+			(at 68.58 158.75 0)
 			(effects
 				(font
@@
 		)
 		(property "Datasheet" ""
-			(at 57.15 168.91 0)
+			(at 68.58 158.75 0)
 			(effects
 				(font
@@
 		)
 		(property "Description" "Power symbol creates a global label with name \"GND\" , ground"
-			(at 57.15 168.91 0)
+			(at 68.58 158.75 0)
 			(effects
 				(font
@@
 		(on_board yes)
 		(dnp no)
-		(fields_autoplaced yes)
 		(property "Reference" "SW2"
-			(at 68.58 158.75 0)
+			(at 83.82 166.37 0)
 			(effects
 				(font
@@
 		)
 		(property "Value" "Reset Button"
-			(at 68.58 161.29 0)
+			(at 83.82 168.91 0)
 			(effects
 				(font
