File: usb2ps2.kicad_sch (KiCad schematic)
At the start: 44 parts, among them CN1 USB, CN2 UART, CN3 PS/2, SW1 Flash Button, SW2 Reset Button, U1 NCP1117-3.3_SOT223, U2 W25Q128JVS, U3 RP2040, Y1 ABM8-272-T3

Commit message: HW Rev 1.2
Parts:
- removed C1, C18, C2, C3: 10u, Capacitor_SMD:C_0805_2012Metric_Pad1.18x1.45mm_HandSolder, symbol Device:C
- removed C10, C11, C12, C13, C14, C17, C6, C7, C8, C9: 100n, Capacitor_SMD:C_0805_2012Metric_Pad1.18x1.45mm_HandSolder, symbol Device:C
- removed C15, C16: 1u, Capacitor_SMD:C_0805_2012Metric_Pad1.18x1.45mm_HandSolder, symbol Device:C
- removed C4, C5: 15p, Capacitor_SMD:C_0805_2012Metric_Pad1.18x1.45mm_HandSolder, symbol Device:C
- removed CN1: USB, LIBS:Medved_USB_Pin4, symbol Connector:Conn_01x04_Pin
- removed CN2: UART, LIBS:Medved_UART_Pin3, symbol Connector:Conn_01x03_Pin
- removed CN3: PS/2, LIBS:Medved_PS2_Con6, symbol Connector:Conn_01x06_Pin
- removed L1, L2: LED, LED_SMD:LED_0805_2012Metric_Pad1.15x1.40mm_HandSolder, symbol Device:LED
- removed PS1: PS/2, LIBS:Connector_Mini-DIN_Female_6Pin_2rows, symbol Connector:Mini-DIN-6
- removed R1, R2: 5.1K, Resistor_SMD:R_0805_2012Metric_Pad1.20x1.40mm_HandSolder, symbol Device:R_Small
- removed R10, R11, R12, R8: 10K, Resistor_SMD:R_0805_2012Metric_Pad1.20x1.40mm_HandSolder, symbol Device:R
- removed R3, R9: 1k, Resistor_SMD:R_0805_2012Metric_Pad1.20x1.40mm_HandSolder, symbol Device:R
- removed R4, R6: 27, Resistor_SMD:R_0805_2012Metric_Pad1.20x1.40mm_HandSolder, symbol Device:R
- removed R5, R7: 1K, Resistor_SMD:R_0805_2012Metric_Pad1.20x1.40mm_HandSolder, symbol Device:R
- removed SW1: Flash Button, LIBS:Button_SMD_3x3x2, symbol Switch:SW_Push_Dual
- removed SW2: Reset Button, LIBS:Button_SMD_3x3x2, symbol Switch:SW_Push_Dual
- removed U1: NCP1117-3.3_SOT223, Package_TO_SOT_SMD:SOT-223-3_TabPin2, symbol Regulator_Linear:NCP1117-3.3_SOT223
- removed U2: W25Q128JVS, Package_SO:SOIC-8_5.23x5.23mm_P1.27mm, symbol Memory_Flash:W25Q128JVS
- removed U3: RP2040, LIBS:RP2040-QFN-56, symbol MCU_RaspberryPi_RP2040:RP2040
- removed USB1: USB_A, Connector_USB:USB_A_CONNFLY_DS1095-WNR0, symbol Connector:USB_A
- removed USB2: USB Type C, LIBS:USB-TYPE-C-31-M-12_lib2, symbol Type-C:HRO-TYPE-C-31-M-12
- removed Y1: ABM8-272-T3, Crystal:Crystal_SMD_3225-4Pin_3.2x2.5mm, symbol Device:Crystal_GND24
- added H1, H2, H3, H4: MountingHole, LIBS:MountingHole_2.1mm, symbol Mechanical:MountingHole
Other:
- removed sheet LS KB_CLK
- removed sheet LS KB_DATA
- removed sheet LS MS_CLK
- removed sheet LS MS_DATA
- added sheet PS2 with Diodes (ps2d.kicad_sch)
- added sheet Power (power.kicad_sch)
- added sheet RP2040 (rp2040.kicad_sch)
- added sheet UART (uart.kicad_sch)
- added sheet USB Stacked (usbstack.kicad_sch)
- note removed: "Crystal"
- note removed: "Flash"
- note removed: "Make sure C10 is close to pin 44 of RP2040"
- note removed: "Make sure C8 is close to pin 45 of RP2040"
- note removed: "Make sure R3 and R4 are close to RP2040"
- note removed: "Power"
