File: power.kicad_sch (KiCad schematic)
At the start: 9 parts, among them CN1 Conn_01x03_Pin, U1 NCP1117-3.3_SOT223

Commit message: HW Rev 1.2 minor fixes
Parts:
- CN1: footprint Connector_PinHeader_2.54mm:PinHeader_1x03_P2.54mm_Vertical -> LIBS:Medved_PinHeader_1x03
Changed lines of the file:
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@@
 			)
 		)
-		(property "Footprint" "Connector_PinHeader_2.54mm:PinHeader_1x03_P2.54mm_Vertical"
+		(property "Footprint" "LIBS:Medved_PinHeader_1x03"
 			(at 143.51 93.98 0)
 			(effects
