File: ps2d.kicad_sch (KiCad schematic)
At the start: 10 parts, among them CN3 PS/2 Pins

Commit message: HW Rev 1.2 minor fixes
Parts:
- CN3: footprint Connector_PinHeader_2.54mm:PinHeader_1x04_P2.54mm_Vertical -> LIBS:Medved_PinHeader_1x04
Changed lines of the file:
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@@
 			)
 		)
-		(property "Footprint" "Connector_PinHeader_2.54mm:PinHeader_1x04_P2.54mm_Vertical"
+		(property "Footprint" "LIBS:Medved_PinHeader_1x04"
 			(at 151.13 85.09 0)
 			(effects
